Commit message: 29/06/21

File: src/BebopS/urdf/multirotor_base.urdf.xacro (robot description, xacro)
@@ -121,5 +121,5 @@
   <xacro:macro name="cam" params="namespace camera_link camera_mass parent *origin *inertia">
     <!-- Camera link -->
-    <link name="camera_box">
+    <link name="camera_link">
       <!--collision>
         <origin xyz="0 0 0" rpy="0 0 0"/>
@@ -142,10 +142,8 @@
     </link>
     <!-- Camera joint with reference to the parent link -->
-    <joint name="camera_joint" type="revolute">
-      <xacro:insert_block name="origin"/>
-      <axis xyz="0 1 0" />
-      <limit effort="1000.0" lower="-3.14" upper="3.14" velocity="0.5"/>
+    <joint name="camera_joint" type="fixed">
       <parent link="${parent}"/>
-      <child link="camera_box"/>
+      <child link="camera_link"/>
+      <origin xyz="0 0 0"   rpy = "0 ${3.1416/2} 0"/>
     </joint>
     <!-- camera
@@ -196,5 +194,5 @@
     </gazebo>
 -->
-<gazebo reference="camera_box">
+<gazebo reference="camera_link">
       <sensor type="camera" name="camera1">
         <update_rate>30.0</update_rate>
@@ -222,5 +220,5 @@
           <imageTopicName>/camera/color/image_raw</imageTopicName>
           <cameraInfoTopicName>camera_info</cameraInfoTopicName>
-          <frameName>camera_box</frameName>
+          <frameName>/camera_link</frameName>
           <hackBaseline>0.07</hackBaseline>
           <distortionK1>0.0</distortionK1>
@@ -233,20 +231,3 @@
     </gazebo>
   </xacro:macro>
-   <!-- This block connects the wheel joint to an actuator (motor), which informs both
-    simulation and visualization of the robot -->
-     <transmission name="camera_trans">
-       <type>transmission_interface/SimpleTransmission</type>
-       <actuator name="$camera_motor">
-         <mechanicalReduction>1</mechanicalReduction>
-       </actuator>
-       <joint name="camera_joint">
-         <hardwareInterface>hardware_interface/PositionJointInterface</hardwareInterface>
-       </joint>
-    </transmission>
-  <!--Gazebo plugin for ROS Control -->
-  <gazebo>
-    <plugin name="gazebo_ros_control2" filename="libgazebo_ros_control.so">
-      <robotNamespace>/</robotNamespace>
-    </plugin>
-  </gazebo>
 </robot>

File: src/ddr/urdf/13-diffdrive.urdf.xacro (robot description, xacro)
@@ -5,5 +5,5 @@
   <xacro:property name="leglen" value="0.6" />
   <xacro:property name="polelen" value="0.2" />
-  <xacro:property name="bodylen" value="0.1" />
+  <xacro:property name="bodylen" value="0.14" />
   <xacro:property name="baselen" value="0.4" />
   <xacro:property name="wheeldiam" value="0.1" />
@@ -28,15 +28,17 @@
     <visual>
       <geometry>
-        <box size="${wheeldiam} ${wheeldiam} ${wheeldiam/2}"/>
+        <box size="${bodylen} ${bodylen} ${bodylen/4}"/>
       </geometry>
-      <material name="blue"/>
     </visual>
     <collision>
       <geometry>
-        <box size="${wheeldiam} ${wheeldiam} ${wheeldiam/2}"/>
+        <box size="${bodylen/2} ${bodylen/2} ${bodylen/4}"/>
       </geometry>
     </collision>
     <xacro:default_inertial mass="50"/>
   </link>
+<gazebo reference="base_link">
+    <material>marker2/diffuce</material>
+</gazebo>
   <xacro:macro name="wheel" params="prefix suffix x y">
     <link name="${prefix}_${suffix}_wheel">
@@ -44,5 +46,6 @@
         <origin xyz="0 0 0" rpy="${pi/2} 0 0" />
         <geometry>
-          <box size="${wheeldiam*0.66} ${wheeldiam*0.66} 0.05"/>
+	  <cylinder radius="${wheeldiam/2}" length="0.04"/>
+          <!--<box size="${wheeldiam*0.66} ${wheeldiam*0.66} 0.05"/>-->
         </geometry>
       </visual>
@@ -50,5 +53,5 @@
         <origin xyz="0 0 0" rpy="${pi/2} 0 0" />
         <geometry>
-          <cylinder radius="${wheeldiam/2}" length="0.1"/>
+          <cylinder radius="${wheeldiam/2}" length="0.04"/>
         </geometry>
       </collision>
@@ -68,5 +71,5 @@
       <kp value="10000000.0" />
       <kd value="1.0" />
-      <material>Gazebo/Grey</material>
+      <material>Gazebo/white</material>
     </gazebo>
     <!-- This block connects the wheel joint to an actuator (motor), which informs both
@@ -88,5 +91,5 @@
   <joint name="camera_joint" type="continuous">
     <axis xyz="0 1 0" />
-    <origin xyz="${camera_link/2 + width} 0 ${bodylen/2}" rpy="0 0 0"/>
+    <origin xyz="${camera_link/2 + width+.05} 0 ${bodylen/2}" rpy="0 0 0"/>
     <parent link="base_link"/>
     <child link="camera_link"/>

Commit message: rrt* drone

File: src/BebopS/urdf/multirotor_base.urdf.xacro (robot description, xacro)
@@ -200,5 +200,5 @@
           <horizontal_fov>1.3962634</horizontal_fov>
           <image>
-            <width>${1920/2}</width>
+            <width>${1080/2}</width>
             <height>${1080/2}</height>
             <format>R8G8B8</format>

File: src/ddr/urdf/diffdrive_kinect.urdf.xacro (robot description, xacro)
@@ -46,5 +46,5 @@
         <origin xyz="0 0 0" rpy="${pi/2} 0 0" />
         <geometry>
-          <cylinder radius="${wheeldiam/2}" length="0.04"/>
+          <cylinder radius="${wheeldiam}" length="0.04"/>
         </geometry>
       </visual>
@@ -147,5 +147,5 @@
 	      <clip>
 		<near>0.1</near>
-		<far>4</far>
+		<far>6</far>
 	      </clip>
 	    </camera>

Commit message: new version

File: src/BebopS/urdf/multirotor_base.urdf.xacro (robot description, xacro)
@@ -121,5 +121,5 @@
   <xacro:macro name="cam" params="namespace camera_link camera_mass parent *origin *inertia">
     <!-- Camera link -->
-    <link name="camera_link">
+    <link name="bebop/camera_link">
       <!--collision>
         <origin xyz="0 0 0" rpy="0 0 0"/>
@@ -144,5 +144,5 @@
     <joint name="camera_joint" type="fixed">
       <parent link="${parent}"/>
-      <child link="camera_link"/>
+      <child link="bebop/camera_link"/>
       <origin xyz="0 0 0"   rpy = "0 ${3.1416/2} 0"/>
     </joint>
@@ -194,5 +194,5 @@
     </gazebo>
 -->
-<gazebo reference="camera_link">
+<gazebo reference="bebop/camera_link">
       <sensor type="camera" name="camera1">
         <update_rate>30.0</update_rate>
@@ -220,5 +220,5 @@
           <imageTopicName>/camera/color/image_raw</imageTopicName>
           <cameraInfoTopicName>camera_info</cameraInfoTopicName>
-          <frameName>/camera_link</frameName>
+          <frameName>/bebop/camera_link</frameName>
           <hackBaseline>0.07</hackBaseline>
           <distortionK1>0.0</distortionK1>

File: src/ddr/urdf/diffdrive_kinect.urdf.xacro (robot description, xacro)
@@ -25,5 +25,5 @@
     </inertial>
   </xacro:macro>
-  <link name="base_link">
+  <link name="ddr/base_link">
     <visual>
       <geometry>
@@ -38,5 +38,5 @@
     <xacro:default_inertial mass="50"/>
   </link>
-  <gazebo reference="base_link">
+  <gazebo reference="ddr/base_link">
     <material>marker2/diffuce</material>
   </gazebo>
@@ -59,5 +59,5 @@
     <joint name="${prefix}_${suffix}_wheel_joint" type="continuous">
       <axis xyz="0 1 0" rpy="0 0 0" />
-      <parent link="base_link"/>
+      <parent link="ddr/base_link"/>
       <child link="${prefix}_${suffix}_wheel"/>
       <origin xyz="${x*0.075} ${y*0.11} -${0.06}" rpy="0 0 0"/>
@@ -96,9 +96,9 @@
     <axis xyz="0 1 0" />
     <origin xyz="${camera_link/2 + width+.05} 0 ${bodylen/2}" rpy="0 0 0"/>
-    <parent link="base_link"/>
-    <child link="camera_link"/>
+    <parent link="ddr/base_link"/>
+    <child link="ddr/camera_link"/>
   </joint>
   <!-- Camera -->
-  <link name="camera_link">
+  <link name="ddr/camera_link">
     <collision>
       <origin xyz="0 0 0" rpy="0 0 0"/>
@@ -135,5 +135,5 @@
   </gazebo>
       <!--camera -->
-    <gazebo reference="camera_link">
+    <gazebo reference="ddr/camera_link">
 	  <sensor name="camera" type="depth">
 	    <update_rate>60</update_rate>
@@ -162,5 +162,5 @@
 	      <depthImageCameraInfoTopicName>/rrbot/camera/depth/camera_info</depthImageCameraInfoTopicName>
 	      <pointCloudTopicName>/rrbot/camera/depth/points</pointCloudTopicName>
-	      <frameName>/camera_link</frameName>
+	      <frameName>/ddr/camera_link</frameName>
 	      <pointCloudCutoff>0.1</pointCloudCutoff>
 	      <pointCloudCutoffMax>4.0</pointCloudCutoffMax>
