Commit message: ddr odom fixed

File: src/ddr/urdf/diffdrive_kinect.urdf.xacro (robot description, xacro)
@@ -7,5 +7,5 @@
   <xacro:property name="bodylen" value="0.1" />
   <xacro:property name="baselen" value="0.4" />
-  <xacro:property name="wheeldiam" value="0.1" />
+  <xacro:property name="wheeldiam" value="0.05" />
   <xacro:property name="pi" value="3.1415" />
   <xacro:property name="camera_link" value=".01" />
@@ -28,5 +28,5 @@
     <visual>
       <geometry>
-        <box size="${wheeldiam} ${wheeldiam} ${wheeldiam/2}"/>
+        <box size="${bodylen} ${bodylen} ${bodylen/2}"/>
       </geometry>
       <material name="blue"/>
@@ -34,5 +34,5 @@
     <collision>
       <geometry>
-        <box size="${wheeldiam} ${wheeldiam} ${wheeldiam/2}"/>
+        <box size="${bodylen} ${bodylen} ${bodylen/2}"/>
       </geometry>
     </collision>
@@ -44,5 +44,5 @@
         <origin xyz="0 0 0" rpy="${pi/2} 0 0" />
         <geometry>
-          <box size="${wheeldiam*0.66} ${wheeldiam*0.66} 0.05"/>
+          <cylinder radius="${wheeldiam}" length="0.02"/>
         </geometry>
       </visual>
@@ -50,5 +50,5 @@
         <origin xyz="0 0 0" rpy="${pi/2} 0 0" />
         <geometry>
-          <cylinder radius="${wheeldiam/2}" length="0.1"/>
+          <cylinder radius="${wheeldiam}" length="0.02"/>
         </geometry>
       </collision>
@@ -150,10 +150,10 @@
 	      <updateRate>0.0</updateRate>
 	      <cameraName>rrbot/camera</cameraName>
-	      <imageTopicName>rrbot/camera/color/image_raw</imageTopicName>
-	      <cameraInfoTopicName>rrbot/camera/color/camera_info</cameraInfoTopicName>
-              <depthImageTopicName>rrbot/camera/depth/image_raw</depthImageTopicName>
-	      <depthImageCameraInfoTopicName>rrbot/camera/depth/camera_info</depthImageCameraInfoTopicName>
-	      <pointCloudTopicName>rrbot/camera/depth/points</pointCloudTopicName>
-	      <frameName>base_correct</frameName>
+	      <imageTopicName>/rrbot/camera/color/image_raw</imageTopicName>
+	      <cameraInfoTopicName>/rrbot/camera/color/camera_info</cameraInfoTopicName>
+              <depthImageTopicName>/rrbot/camera/depth/image_raw</depthImageTopicName>
+	      <depthImageCameraInfoTopicName>/rrbot/camera/depth/camera_info</depthImageCameraInfoTopicName>
+	      <pointCloudTopicName>/rrbot/camera/depth/points</pointCloudTopicName>
+	      <frameName>camera_link</frameName>
 	      <pointCloudCutoff>0.1</pointCloudCutoff>
 	      <pointCloudCutoffMax>6.0</pointCloudCutoffMax>

Commit message: occupacy grid fixed, incomplete rrt

File: src/ddr/urdf/diffdrive_kinect.urdf.xacro (robot description, xacro)
@@ -88,5 +88,5 @@
   <joint name="camera_joint" type="continuous">
     <axis xyz="0 1 0" />
-    <origin xyz="${camera_link/2 + width} 0 ${bodylen/2}" rpy="0 0 0"/>
+    <origin xyz="${camera_link/2 + width} 0 ${bodylen/2+.07}" rpy="0 0 0"/>
     <parent link="base_link"/>
     <child link="camera_link"/>
@@ -140,5 +140,5 @@
 	      <clip>
 		<near>0.1</near>
-		<far>6</far>
+		<far>4</far>
 	      </clip>
 	    </camera>
@@ -157,5 +157,5 @@
 	      <frameName>/camera_link</frameName>
 	      <pointCloudCutoff>0.1</pointCloudCutoff>
-	      <pointCloudCutoffMax>6.0</pointCloudCutoffMax>
+	      <pointCloudCutoffMax>4.0</pointCloudCutoffMax>
 	      <distortionK1>0</distortionK1>
 	      <distortionK2>0</distortionK2>

Commit message: RRT* Firts try

File: src/ddr/urdf/diffdrive_kinect.urdf.xacro (robot description, xacro)
@@ -37,5 +37,5 @@
       </geometry>
     </collision>
-    <xacro:default_inertial mass="50"/>
+    <xacro:default_inertial mass="100"/>
   </link>
   <xacro:macro name="wheel" params="prefix suffix x y">
@@ -44,5 +44,5 @@
         <origin xyz="0 0 0" rpy="${pi/2} 0 0" />
         <geometry>
-          <cylinder radius="${wheeldiam}" length="0.02"/>
+          <cylinder radius="${wheeldiam}" length="0.04"/>
         </geometry>
       </visual>
@@ -50,8 +50,8 @@
         <origin xyz="0 0 0" rpy="${pi/2} 0 0" />
         <geometry>
-          <cylinder radius="${wheeldiam}" length="0.02"/>
+          <cylinder radius="${wheeldiam}" length="0.04"/>
         </geometry>
       </collision>
-      <xacro:default_inertial mass="50"/>
+      <xacro:default_inertial mass="100"/>
     </link>
     <joint name="${prefix}_${suffix}_wheel_joint" type="continuous">
@@ -64,8 +64,13 @@
     physical properties. See http://gazebosim.org/tutorials/?tut=ros_urdf for more-->
     <gazebo reference="${prefix}_${suffix}_wheel">
-      <mu1 value="200.0"/>
-      <mu2 value="100.0"/>
+      <mu1 value="2000.0"/>
+      <mu2 value="1000.0"/>
       <kp value="10000000.0" />
-      <kd value="1.0" />
+      <kd value="1000000000.0" />
+      <contact>
+          <ode>
+            <min_depth>0.5</min_depth>
+          </ode>
+        </contact>
       <material>Gazebo/Grey</material>
     </gazebo>

Commit message: state machine 1

File: src/ddr/urdf/diffdrive_kinect.urdf.xacro (robot description, xacro)
@@ -5,5 +5,5 @@
   <xacro:property name="leglen" value="0.6" />
   <xacro:property name="polelen" value="0.2" />
-  <xacro:property name="bodylen" value="0.1" />
+  <xacro:property name="bodylen" value="0.14" />
   <xacro:property name="baselen" value="0.4" />
   <xacro:property name="wheeldiam" value="0.05" />
@@ -30,13 +30,15 @@
         <box size="${bodylen} ${bodylen} ${bodylen/2}"/>
       </geometry>
-      <material name="blue"/>
     </visual>
     <collision>
       <geometry>
-        <box size="${bodylen} ${bodylen} ${bodylen/2}"/>
+         <box size="${bodylen/2} ${bodylen/2} ${bodylen/4}"/>
       </geometry>
     </collision>
-    <xacro:default_inertial mass="100"/>
+    <xacro:default_inertial mass="50"/>
   </link>
+  <gazebo reference="base_link">
+    <material>marker2/diffuce</material>
+  </gazebo>
   <xacro:macro name="wheel" params="prefix suffix x y">
     <link name="${prefix}_${suffix}_wheel">
@@ -44,5 +46,5 @@
         <origin xyz="0 0 0" rpy="${pi/2} 0 0" />
         <geometry>
-          <cylinder radius="${wheeldiam}" length="0.04"/>
+          <cylinder radius="${wheeldiam/2}" length="0.04"/>
         </geometry>
       </visual>
@@ -93,5 +95,5 @@
   <joint name="camera_joint" type="continuous">
     <axis xyz="0 1 0" />
-    <origin xyz="${camera_link/2 + width} 0 ${bodylen/2+.07}" rpy="0 0 0"/>
+    <origin xyz="${camera_link/2 + width+.05} 0 ${bodylen/2}" rpy="0 0 0"/>
     <parent link="base_link"/>
     <child link="camera_link"/>

Commit message: update 23/05/22

File: src/ddr/urdf/diffdrive_kinect.urdf.xacro (robot description, xacro)
@@ -25,9 +25,13 @@
     </inertial>
   </xacro:macro>
+<link name="dummy">
+   </link>
   <link name="ddr/base_link">
     <visual>
+	<origin rpy="0 0 0" xyz="0 0 -.03"/>
       <geometry>
-        <box size="${bodylen} ${bodylen} ${bodylen/2}"/>
-      </geometry>
+          <mesh filename="package://ddr/urdf/caja_1.dae"/>
+          <!-- <box size="${body_width} ${body_width} ${body_height}"/> --> <!-- [m] [m] [m] -->
+        </geometry>
     </visual>
     <collision>
@@ -38,4 +42,8 @@
     <xacro:default_inertial mass="50"/>
   </link>
+<joint name="dummy_joint" type="fixed">
+     <parent link="dummy"/>
+     <child link="ddr/base_link"/>
+   </joint>
   <gazebo reference="ddr/base_link">
     <material>marker2/diffuce</material>
@@ -44,7 +52,8 @@
     <link name="${prefix}_${suffix}_wheel">
       <visual>
-        <origin xyz="0 0 0" rpy="${pi/2} 0 0" />
+        <origin xyz="0 0 0" rpy="${-pi/2} 0 0 " />
         <geometry>
-          <cylinder radius="${wheeldiam}" length="0.04"/>
+	 <cylinder radius="${wheeldiam}" length="0.04"/>
+          <!--<mesh filename="package://ddr/urdf/llanta.dae"/> -->
         </geometry>
       </visual>
@@ -94,5 +103,5 @@
   <xacro:wheel prefix="right" suffix="back" x="-1" y="-1"/>
   <joint name="camera_joint" type="continuous">
-    <axis xyz="0 1 0" />
+    <axis xyz="1 0 0" />
     <origin xyz="${camera_link/2 + width+.05} 0 ${bodylen/2}" rpy="0 0 0"/>
     <parent link="ddr/base_link"/>
